File: Switch Machine PCB/SMRRC_Switch.kicad_pcb (KiCad board)
At the start: 2 copper layers, 98 x 68 mm, 70 parts, among them J1 Conn_01x05, J10 Conn_01x04, J2 Conn_01x03, J3 Conn_01x03, J4 Conn_01x08_Socket, J5 Conn_01x06, J6 Conn_01x04, J7 Conn_01x04, J8 Conn_01x04, J9 Conn_01x04, K1 J114AF, SW1 SW_Push, SW2 SW_Push, U1 L78L05_SOT89, U10 SSM6N7002CFU, U11 SSM6N7002CFU, U12 SSM6N7002CFU, U13 SSM6N7002CFU, U14 SSM6N7002CFU, U2 L7806, U3 PIC16F15345-I/SO, U4 THVD1500, U5 SN74HC259DR, U6 SN74HC259DR, U7 SSM6N7002CFU, U8 SSM6N7002CFU, U9 SSM6N7002CFU

Commit message: SwitchMachinePCB
Parts:
- removed C10, C11: 0.1uf, Capacitor_SMD:C_0805_2012Metric_Pad1.18x1.45mm_HandSolder
- removed J10, J6, J7, J8, J9: Conn_01x04, TerminalBlock_Phoenix:TerminalBlock_Phoenix_PT-1,5-4-3.5-H_1x04_P3.50mm_Horizontal
- removed R14, R15, R16, R17, R18, R19, R20, R21: 1K0, Resistor_THT:R_Axial_DIN0204_L3.6mm_D1.6mm_P7.62mm_Horizontal
- removed U10, U11, U12, U13, U14, U7, U8, U9: SSM6N7002CFU, Package_TO_SOT_SMD:SOT-363_SC-70-6_Handsoldering
- removed U5, U6: SN74HC259DR, Package_SO:SOIC-16W_5.3x10.2mm_P1.27mm
- added D8: 1N4148W, Diode_SMD:D_SOD-123, F.Cu at (121.6, 103.5)
- added Q1: 2N3906, Package_TO_SOT_THT:TO-92_Inline, F.Cu at (131.7, 105.1)
- added Q2: 2N3904, Package_TO_SOT_THT:TO-92_Inline, F.Cu at (131.7, 100.1)
- added Q3: 2N3904, Package_TO_SOT_THT:TO-92_Inline, F.Cu at (131.7, 95.0)
- J5: value Conn_01x06 -> Molex 3x4 10181120; footprint TerminalBlock_MetzConnect:TerminalBlock_MetzConnect_Type059_RT06306HBWC_1x06_P3.50mm_Horizontal -> Molex10181201:Molex10181120
- R10, R11, R8, R9: value 1K0 -> 10K; footprint Resistor_THT:R_Axial_DIN0204_L3.6mm_D1.6mm_P7.62mm_Horizontal -> Resistor_SMD:R_0805_2012Metric_Pad1.20x1.40mm_HandSolder
- R12, R13: value 1K0 -> 2K2; footprint Resistor_THT:R_Axial_DIN0204_L3.6mm_D1.6mm_P7.62mm_Horizontal -> Resistor_SMD:R_0805_2012Metric_Pad1.20x1.40mm_HandSolder
- R7: value 1K0 -> 4K7; footprint Resistor_THT:R_Axial_DIN0204_L3.6mm_D1.6mm_P7.62mm_Horizontal -> Resistor_SMD:R_0805_2012Metric_Pad1.20x1.40mm_HandSolder
- moved SW1 60.7 mm to (96.3, 94.6), turned to 0 degrees
- moved D4 56.2 mm to (96.3, 99.6), turned to 180 degrees
- moved SW2 50.4 mm to (107.3, 94.6), turned to 0 degrees
- moved R3 49.8 mm to (101.3, 100.6), turned to 90 degrees
- moved J2 45.2 mm to (97.0, 104.6)
- moved D5 44.8 mm to (107.3, 99.6), turned to 180 degrees
- moved R2 41.7 mm to (106.3, 103.6), turned to 90 degrees
- moved R4 39.7 mm to (108.3, 103.6), turned to 90 degrees
- moved R5 39.4 mm to (112.3, 100.6), turned to 90 degrees
- moved J5 26.7 mm to (146.1, 106.6)
- moved R7 23.3 mm to (128.3, 106.0), turned to 180 degrees
- moved R9 19.0 mm to (128.3, 108.6), turned to 180 degrees
- moved R8 18.6 mm to (128.3, 103.5), turned to 180 degrees
- moved H2 13.7 mm to (155.6, 91.4)
- moved H1 13.4 mm to (67.9, 91.4)
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Connections:
- J5 pad 1: 1N -> +12V
- J5 pad 2: 1C -> GND
- J5 pad 3: 1R -> Net-(D8-K)
- J5 pad 4: 2N -> Net-(J5-Pin_4)
- J5 pad 5: 2C -> Net-(J5-Pin_5)
- J5 pad 6: 2R -> unconnected-(J5-Pin_6-Pad6)
- R10 pad 1: Net-(U8-D2) -> Net-(Q3-B)
- R10 pad 2: Net-(J7-Pin_2) -> GND
- R11 pad 1: Net-(U9-D1) -> Net-(Q2-B)
- R11 pad 2: Net-(J7-Pin_3) -> GND
- R12 pad 1: Net-(U9-D2) -> Net-(U3-RC1)
- R12 pad 2: Net-(J7-Pin_4) -> Net-(Q2-B)
- R13 pad 1: Net-(U10-D1) -> Net-(U3-RC2)
- R13 pad 2: Net-(J8-Pin_2) -> Net-(Q3-B)
- R7 pad 2: Net-(J6-Pin_2) -> Net-(D8-A)
- R8 pad 1: Net-(U7-D2) -> +5V
- R8 pad 2: Net-(J6-Pin_3) -> Net-(D8-A)
- R9 pad 1: Net-(U8-D1) -> Net-(Q1-C)
- R9 pad 2: Net-(J6-Pin_4) -> GND
- U3 pad 16: Net-(U3-RC0) -> Net-(Q1-C)
- U3 pad 6: Net-(U3-RC4) -> unconnected-(U3-RC4-Pad6)
- U3 pad 7: Net-(U3-RC3) -> unconnected-(U3-RC3-Pad7)
- U3 pad 8: Net-(U3-RC6) -> unconnected-(U3-RC6-Pad8)
- U3 pad 9: Net-(U3-RC7) -> unconnected-(U3-RC7-Pad9)
Routing:
- net +12V: track 252.2 -> 157.7 mm
- net K1: track 86.9 -> 10.9 mm, vias 2 -> 0
- net Net-(U3-RC7): track 52.9 -> 0.00 mm, vias 3 -> 0
- net Net-(U3-RC6): track 49.7 -> 0.00 mm, vias 3 -> 0
- net GND: track 473.7 -> 430.3 mm, vias 21 -> 6
- net Net-(U3-RC0): track 40.1 -> 0.00 mm, vias 3 -> 0
- net Net-(J2-Pin_1): track 72.8 -> 37.7 mm, vias 1 -> 0
- net Net-(U14-G1): track 34.7 -> 0.00 mm, vias 2 -> 0
- net Net-(U14-G2): track 29.8 -> 0.00 mm, vias 2 -> 0
- net Net-(U3-RC3): track 29.1 -> 0.00 mm, vias 2 -> 0
- net Net-(U10-G1): track 27.1 -> 0.00 mm, vias 2 -> 0
- net +5V: track 198.0 -> 171.2 mm, vias 10 -> 9
- net Net-(J2-Pin_3): track 67.2 -> 42.7 mm
- net Net-(U10-G2): track 24.1 -> 0.00 mm, vias 2 -> 0
- net Net-(U3-RC1): track 42.3 -> 18.4 mm, vias 3 -> 2
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Other:
- board size 98 x 68 mm -> 95.4 x 54.4 mm
- board text added: "Serial Model Railroad Control DMFE 2026 Rev. n/c"
- board text added: "Switch Machine"
- board text removed: "2R 2C 2N 1R 1C 1N"
- board text removed: "COM GRN YEL RED"
- board text removed: "Serial Model Railroad Control DMFE 2025 Rev. n/c"
- board text removed: "Switch And Signal"

Commit message: Switch machine PCB done
Parts:
- added D9: 1N4148W, Diode_SMD:D_SOD-123, F.Cu at (121.5, 103.0)
- added Q4: 2N3906, Package_TO_SOT_THT:TO-92_Inline, F.Cu at (133.2, 107.1)
- added Q5: 2N7000, Package_TO_SOT_THT:TO-92_Inline, F.Cu at (122.7, 138.6)
- added R14: 10K, Resistor_SMD:R_0805_2012Metric_Pad1.20x1.40mm_HandSolder, F.Cu at (129.8, 107.7)
- added R15: 4K7, Resistor_SMD:R_0805_2012Metric_Pad1.20x1.40mm_HandSolder, F.Cu at (129.8, 105.7)
- added R16: 10K, Resistor_SMD:R_0805_2012Metric_Pad1.20x1.40mm_HandSolder, F.Cu at (129.8, 109.7)
- added R17: 27K, Resistor_SMD:R_0805_2012Metric_Pad1.20x1.40mm_HandSolder, F.Cu at (119.1, 136.8)
- added R18: 10K, Resistor_SMD:R_0805_2012Metric_Pad1.20x1.40mm_HandSolder, F.Cu at (119.1, 138.9)
- moved R7 6.63 mm to (129.8, 99.6)
- moved R9 5.16 mm to (129.8, 103.7)
- moved D8 4.70 mm to (121.5, 98.8)
- moved R11 3.72 mm to (129.8, 97.6)
- moved R12 3.27 mm to (129.8, 95.5)
- moved Q1 3.25 mm to (133.2, 102.3)
- moved Q2 3.04 mm to (133.2, 97.4)
- moved R10 2.93 mm to (129.8, 93.4)
- moved Q3 2.83 mm to (133.2, 92.6)
- moved R13 2.61 mm to (129.8, 91.2)
- moved R8 2.41 mm to (129.8, 101.6)
Connections:
- D6 pad 2: K1 -> Net-(D6-A)
- D7 pad 1: K1 -> Net-(D6-A)
- J5 pad 6: unconnected-(J5-Pin_6-Pad6) -> Net-(D9-K)
- K1 pad A2: K1 -> Net-(D6-A)
- R3 pad 2: Net-(J2-Pin_1) -> StatLED1
- R5 pad 2: Net-(J2-Pin_3) -> StatLED2
- U3 pad 6: unconnected-(U3-RC4-Pad6) -> StatLED2
- U3 pad 7: unconnected-(U3-RC3-Pad7) -> StatLED1
- U3 pad 8: unconnected-(U3-RC6-Pad8) -> Net-(Q4-C)
- U3 pad 9: unconnected-(U3-RC7-Pad9) -> K1
Routing:
- net GND: track 430.3 -> 394.5 mm, vias 6 -> 8
- net +5V: track 171.2 -> 138.3 mm, vias 9 -> 5
- net Net-(Q4-C): track 0.00 -> 29.8 mm, vias 0 -> 3
- net Net-(D9-K): track 0.00 -> 24.7 mm, vias 0 -> 1
- net StatLED1: track 0.00 -> 24.3 mm
- net StatLED2: track 0.00 -> 22.4 mm
- net K1: track 10.9 -> 28.5 mm
- net Net-(D6-A): track 0.00 -> 17.1 mm
- net Net-(Q1-C): track 17.2 -> 28.1 mm, vias 2 -> 3
- net Net-(J2-Pin_3): track 42.7 -> 32.7 mm
- net Net-(D9-A): track 0.00 -> 9.14 mm, vias 0 -> 2
- net Net-(Q5-G): track 0.00 -> 8.62 mm
- net Net-(Q4-B): track 0.00 -> 4.78 mm, vias 0 -> 1
- net Net-(U3-RC1): track 18.4 -> 22.8 mm
- net Net-(U3-RC2): track 24.3 -> 27.7 mm
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