File: Switch Machine PCB/SMRRC_Switch.kicad_sch (KiCad schematic)
At the start: 49 parts, among them J1 Conn_01x05, J2 Conn_01x03, J3 Conn_01x03, J4 Conn_01x08_Socket, J5 Molex 3x4 10181120, K1 J114AF, Q1 2N3906, Q2 2N3904, Q3 2N3904, SW1 SW_Push, SW2 SW_Push, U1 L78L05_SOT89, U2 L7806, U3 PIC16F15345-I/SO, U4 THVD1500

Commit message: SwitchMachinePCB
Parts:
- J5: footprint (none) -> Molex10181201:Molex10181120
Changed lines of the file:
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@@
 			)
 		)
-		(property "Footprint" ""
+		(property "Footprint" "Molex10181201:Molex10181120"
 			(at 222.25 64.77 0)
 			(hide yes)

Commit message: Switch machine PCB done
Parts:
- added D9: 1N4148W, Diode_SMD:D_SOD-123, symbol Diode:1N4148W
- added Q4: 2N3906, Package_TO_SOT_THT:TO-92_Inline, symbol Transistor_BJT:2N3906
- added Q5: 2N7000, Package_TO_SOT_THT:TO-92_Inline, symbol Transistor_FET:2N7000
- added R14, R16, R18: 10K, Resistor_SMD:R_0805_2012Metric_Pad1.20x1.40mm_HandSolder, symbol Device:R_Small
- added R15: 4K7, Resistor_SMD:R_0805_2012Metric_Pad1.20x1.40mm_HandSolder, symbol Device:R_Small
- added R17: 27K, Resistor_SMD:R_0805_2012Metric_Pad1.20x1.40mm_HandSolder, symbol Device:R_Small
Connections:
- net +5V: now also Q4.1 (E), R14.1
- net GND: now also Q5.1 (S), R16.2, R17.2
- net K1: now also U3.9 (RC7), R18.1; no longer D6.2 (A), D7.1 (K), K1.A2
- net at J2.1 (Pin_1), R2.2, SW1.2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: no longer R3.2
- net at J2.3 (Pin_3), R4.2, SW2.2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: no longer R5.2
- net StatLED2: now reaches U3.6 (RC4)
- net StatLED2: now also R5.2
- net StatLED1: now reaches U3.7 (RC3)
- net StatLED1: now also R3.2
- net at U3.8 (RC6): now also Q4.3 (C), R16.1
- net at J5.6 (Pin_6): now also D9.1 (K)
- new net: Q4.2 (B), R15.1
- new net: D6.2 (A), D7.1 (K), K1.A2, Q5.3 (D)
- new net: Q5.2 (G), R17.1, R18.2
- new net: D9.2 (A), R14.2, R15.2
- no-connect marks 5 -> 0
Other:
- note added: "+12V GND Control Feedback N Feedback R Control 2 1N 1C 1R 2N 2C 2R"
- note added: "This board sits on the RS485 bus and controls one switch machine."
- note removed: "+12V GND Control Feedback N Feedback R ?? 1N 1C 1R 2N 2C 2R"
