File: Block Relay PCB/BlockRelay.kicad_sch (KiCad schematic)
At the start: 86 parts, among them J1 Screw_Terminal_01x16, J2 Conn_02x06_Odd_Even, J3 Conn_02x08_Odd_Even, K1 Relay_DPDT, K2 Relay_DPDT, K3 Relay_DPDT, K4 Relay_DPDT, K5 Relay_DPDT, K6 Relay_DPDT, Q1 2N7000, Q2 2N7000, Q3 2N7000, Q4 2N7000, Q5 2N7000, Q6 2N7000, U1 74HC259, U2 74LS251, U5 L78L05_SOT89

Commit message: worked on block relay pcb
Parts:
- added D28, D29, D30, D31: Yellow LED, LED_SMD:LED_1206_3216Metric_Pad1.42x1.75mm_HandSolder, symbol Device:LED_Small_Filled
- added H10, H7, H8, H9: MountingHole, MountingHole:MountingHole_3.2mm_M3, symbol Mechanical:MountingHole
- added R20, R22, R24, R26: 27K, Resistor_SMD:R_0805_2012Metric_Pad1.20x1.40mm_HandSolder, symbol Device:R_Small
- added R21, R23, R25, R27: 2K2, Resistor_SMD:R_0805_2012Metric_Pad1.20x1.40mm_HandSolder, symbol Device:R_Small
- J2: footprint Connector_PinSocket_2.54mm:PinSocket_2x06_P2.54mm_Vertical -> Connector_PinHeader_2.54mm:PinHeader_2x06_P2.54mm_Vertical
Connections:
- net +5V: now also D28.2 (A), D29.2 (A), D30.2 (A), D31.2 (A), R20.1, R22.1, R24.1, R26.1
- net Blk1: no longer K4.12
- net Blk2: now also K4.12
- net at J3.16 (Pin_16), U2.1 (I3): now also R27.2
- net at J3.14 (Pin_14), U2.2 (I2): now also R25.2
- net at J3.12 (Pin_12), U2.3 (I1): now also R23.2
- net at J3.10 (Pin_10), U2.4 (I0): now also R21.2
- new net: D28.1 (K), R20.2, R21.1
- new net: D31.1 (K), R26.2, R27.1
- new net: D30.1 (K), R24.2, R25.1
- new net: D29.1 (K), R22.2, R23.1
Other:
- note added: "Block 1 North Rail"
- note added: "Block 1 South Rail"
- note added: "Block 2 North Rail"
- note added: "Block 2 South Rail"
- note added: "Block Detection Module Quad Detector w/ OC Output"
- note removed: "Block Detection Module Quad Detector w/ TTL Output"

Commit message: Block Relay ready to print
Parts:
- removed C16, C4, C5, C7: 0.1uF, Capacitor_SMD:C_0805_2012Metric_Pad1.18x1.45mm_HandSolder, symbol Device:C_Small
- removed D22, D23, D25, D27: Schottky_AKA DPAK, Package_TO_SOT_SMD:TO-252-2, symbol Device:D_Schottky_AKA
- removed D29, D31: Yellow LED, LED_SMD:LED_1206_3216Metric_Pad1.42x1.75mm_HandSolder, symbol Device:LED_Small_Filled
- removed H7, H8: MountingHole, MountingHole:MountingHole_3.2mm_M3, symbol Mechanical:MountingHole
- removed J1: Screw_Terminal_01x16, TerminalBlock_Phoenix:TerminalBlock_Phoenix_PT-1,5-16-3.5-H_1x16_P3.50mm_Horizontal, symbol Connector:Screw_Terminal_01x16
- removed J3: Conn_02x08_Odd_Even, Connector_PinSocket_2.54mm:PinSocket_2x08_P2.54mm_Vertical, symbol Connector_Generic:Conn_02x08_Odd_Even
- removed R17, R19: 1K0, Resistor_SMD:R_0805_2012Metric_Pad1.20x1.40mm_HandSolder, symbol Device:R_Small
- removed R22, R26: 27K, Resistor_SMD:R_0805_2012Metric_Pad1.20x1.40mm_HandSolder, symbol Device:R_Small
- removed R23, R27: 2K2, Resistor_SMD:R_0805_2012Metric_Pad1.20x1.40mm_HandSolder, symbol Device:R_Small
- removed U2: 74LS251, Package_SO:SO-16_3.9x9.9mm_P1.27mm, symbol 74xx:74LS251
- added J1: Screw_Terminal_01x12, TerminalBlock_Phoenix:TerminalBlock_Phoenix_PT-1,5-12-3.5-H_1x12_P3.50mm_Horizontal, symbol Connector:Screw_Terminal_01x12
- added J3: Conn_02x05_Odd_Even, Connector_PinSocket_2.54mm:PinSocket_2x05_P2.54mm_Vertical, symbol Connector_Generic:Conn_02x05_Odd_Even
- renumbered C12 to C10, C10 to C11, C13 to C12, C11 to C13, C6 to C2, C15 to C3, C2 to C4, C3 to C5, D14 to D10, D2 to D11, D17 to D12, D8 to D13, D5 to D14, D11 to D15, D15 to D16, D4 to D17, D10 to D19, D20 to D2, D7 to D20, D13 to D21, D16 to D22, D6 to D23, D19 to D24, D12 to D25, D24 to D3, D21 to D4, D26 to D5, D28 to D6, D30 to D7, D3 to D8, H10 to H1, H9 to H2, H1 to H3, H2 to H4, H3 to H6, H6 to H7, H4 to H8, K4 to K2, K2 to K3, K5 to K4, K3 to K5, Q4 to Q2, Q2 to Q3, Q5 to Q4, Q3 to Q5, R16 to R1, R13 to R11, R3 to R12, R6 to R13, R11 to R14, R14 to R15, R4 to R16, R7 to R17, R12 to R18, R15 to R19, R18 to R2, R9 to R20, R8 to R21, R20 to R3, R21 to R4, R24 to R5, R1 to R6, R25 to R7, R2 to R8, R5 to R9, U5 to U1, U1 to U2
Connections:
- net +12V: now also J1.1 (Pin_1), J1.2 (Pin_2), J3.2 (Pin_2), J3.4 (Pin_4)
- net Blk1: now also J3.1 (Pin_1)
- net Blk2: now also J3.5 (Pin_5)
- net Det12V: now also J1.5 (Pin_5)
- net GND: now also J1.3 (Pin_3), J1.4 (Pin_4), J3.6 (Pin_6), J3.8 (Pin_8)
- net Thr1: now also J1.6 (Pin_6)
- net Thr2: now also J1.7 (Pin_7)
- net Thr3: now also J1.8 (Pin_8)
- net at C3.1, D3.2 (K), D5.1 (A)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: now also J1.11 (Pin_11), J3.7 (Pin_7)
- net at R4.2: now also J1.10 (Pin_10), J3.9 (Pin_9)
- net at C2.1, D2.2 (K), D4.1 (A)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: now also J1.9 (Pin_9), J3.3 (Pin_3)
- net at R7.2: now also J1.12 (Pin_12), J3.10 (Pin_10)
- net A3: no longer names the net of J2.8 (Pin_8)
- net A4: no longer names the net of J2.9 (Pin_9)
- net nE1: no longer names the net of J2.10 (Pin_10)
- net nE1: no longer U2.14 (E)
- net nE2 renamed nE
- net nE: now also U2.14 (E)
- no-connect marks 10 -> 17
Other:
- note added: "+12 +12 GND GND Det12V Thr1 Thr2 Thr3 Blk1NR Blk1Det Blk2NR Blk2Det"
- note removed: "+12 +12 GND GND TrkGND Det12V Thr1 Thr2 Thr3 Blk1NR Blk1SR Blk2NR Blk2SR"
- note removed: "Block 1 South Rail"
- note removed: "Block 2 South Rail"
- moved on the sheet: D6, D7, R3, R4, R5, R7
